File: liquids/PCB/InstrumentationAmp/src/InstrumentationAmplifier.sch (EAGLE design)
At the start: 21 parts, among them U1 LM317AEMP/NOPB, U2 LM337IMP/NOPB, U3 ADA4177-4ARZ-R7R_14_ADI-M

Commit message: Added pin headers for regualted output
Parts:
- JP2: device pinhead:PINHD-1X2 -> pinhead:PINHD-1X55X2MM
Connections:
- net GND: now also JP2.4
- net IN+: now also JP2.2; no longer JP2.1
- net IN-: now also JP2.3; no longer JP2.2
- net VREG+: now also JP2.1
- net VREG-: now also JP2.5
Changed lines of the file:
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@@
 <part name="AR3-" library="rcl" library_urn="urn:adsk.eagle:library:334" deviceset="R-US_" device="R0603" package3d_urn="urn:adsk.eagle:package:23555/3" value="1k"/>
 <part name="U3" library="OpAmpADA4177-4" deviceset="ADA4177-4ARZ-R7" device="R_14_ADI-M"/>
-<part name="JP2" library="pinhead" library_urn="urn:adsk.eagle:library:325" deviceset="PINHD-1X2" device="" package3d_urn="urn:adsk.eagle:package:22435/2"/>
 <part name="VR3" library="ST4ETB502" deviceset="ST4ETB502" device=""/>
 <part name="AR3+" library="rcl" library_urn="urn:adsk.eagle:library:334" deviceset="R-US_" device="R0603" package3d_urn="urn:adsk.eagle:package:23555/3" value="1k"/>
@@
 <part name="JP3" library="pinhead" library_urn="urn:adsk.eagle:library:325" deviceset="PINHD-1X2" device="" package3d_urn="urn:adsk.eagle:package:22435/2"/>
 <part name="GND11" library="supply1" library_urn="urn:adsk.eagle:library:371" deviceset="GND" device=""/>
+<part name="JP2" library="pinhead" library_urn="urn:adsk.eagle:library:325" deviceset="PINHD-1X5" device="5X2MM" package3d_urn="urn:adsk.eagle:package:22466/2"/>
+<part name="GND12" library="supply1" library_urn="urn:adsk.eagle:library:371" deviceset="GND" device=""/>
 </parts>
 <sheets>
@@
 <attribute name="VALUE" x="22.86" y="20.32" size="1.778" layer="96"/>
 </instance>
-<instance part="GND7" gate="1" x="40.64" y="27.94" smashed="yes" rot="R90">
-<attribute name="VALUE" x="43.18" y="25.4" size="1.778" layer="96" rot="R90"/>
-</instance>
-<instance part="GND8" gate="1" x="35.56" y="33.02" smashed="yes" rot="R90">
-<attribute name="VALUE" x="38.1" y="30.48" size="1.778" layer="96" rot="R90"/>
+<instance part="GND7" gate="1" x="38.1" y="22.86" smashed="yes" rot="R90">
+<attribute name="VALUE" x="40.64" y="20.32" size="1.778" layer="96" rot="R90"/>
+</instance>
+<instance part="GND8" gate="1" x="35.56" y="38.1" smashed="yes" rot="R90">
+<attribute name="VALUE" x="38.1" y="35.56" size="1.778" layer="96" rot="R90"/>
 </instance>
 <instance part="GND9" gate="1" x="30.48" y="30.48" smashed="yes" rot="R90">
@@
 <attribute name="VALUE" x="180.0606" y="57.3786" size="2.0828" layer="96" ratio="6" rot="SR0"/>
 </instance>
-<instance part="JP2" gate="G$1" x="132.08" y="78.74" smashed="yes" rot="R90">
-<attribute name="NAME" x="126.365" y="72.39" size="1.778" layer="95" rot="R90"/>
-<attribute name="VALUE" x="137.16" y="72.39" size="1.778" layer="96" rot="R90"/>
-</instance>
 <instance part="VR3" gate="G$1" x="111.76" y="25.4" smashed="yes" rot="R90">
 <attribute name="NAME" x="104.14" y="41.91" size="1.778" layer="95" rot="R90" align="center-left"/>
@@
 <instance part="GND11" gate="1" x="246.38" y="40.64" smashed="yes" rot="R270">
 <attribute name="VALUE" x="243.84" y="43.18" size="1.778" layer="96" rot="R270"/>
+</instance>
+<instance part="JP2" gate="A" x="132.08" y="86.36" smashed="yes" rot="R90">
+<attribute name="NAME" x="123.825" y="80.01" size="1.778" layer="95" rot="R90"/>
+<attribute name="VALUE" x="142.24" y="80.01" size="1.778" layer="96" rot="R90"/>
+</instance>
+<instance part="GND12" gate="1" x="137.16" y="73.66" smashed="yes">
+<attribute name="VALUE" x="134.62" y="71.12" size="1.778" layer="96"/>
 </instance>
 </instances>
@@
 <segment>
 <pinref part="GND9" gate="1" pin="GND"/>
-<pinref part="GND8" gate="1" pin="GND"/>
-<pinref part="JP1" gate="A" pin="2"/>
-<wire x1="7.62" y1="33.02" x2="33.02" y2="33.02" width="0.1524" layer="91"/>
 <pinref part="JP1" gate="A" pin="3"/>
 <wire x1="7.62" y1="30.48" x2="27.94" y2="30.48" width="0.1524" layer="91"/>
-</segment>
-<segment>
-<pinref part="JP1" gate="A" pin="4"/>
-<pinref part="GND7" gate="1" pin="GND"/>
-<wire x1="7.62" y1="27.94" x2="38.1" y2="27.94" width="0.1524" layer="91"/>
 </segment>
 <segment>
@@
 <pinref part="GND11" gate="1" pin="GND"/>
 <wire x1="248.92" y1="43.18" x2="248.92" y2="40.64" width="0.1524" layer="91"/>
+</segment>
+<segment>
+<pinref part="JP2" gate="A" pin="4"/>
+<wire x1="134.62" y1="83.82" x2="134.62" y2="76.2" width="0.1524" layer="91"/>
+<pinref part="GND12" gate="1" pin="GND"/>
+<wire x1="134.62" y1="76.2" x2="137.16" y2="76.2" width="0.1524" layer="91"/>
+</segment>
+<segment>
+<pinref part="JP1" gate="A" pin="2"/>
+<wire x1="7.62" y1="33.02" x2="27.94" y2="33.02" width="0.1524" layer="91"/>
+<wire x1="27.94" y1="33.02" x2="27.94" y2="38.1" width="0.1524" layer="91"/>
+<pinref part="GND8" gate="1" pin="GND"/>
+<wire x1="27.94" y1="38.1" x2="33.02" y2="38.1" width="0.1524" layer="91"/>
+</segment>
+<segment>
+<pinref part="JP1" gate="A" pin="4"/>
+<wire x1="7.62" y1="27.94" x2="27.94" y2="27.94" width="0.1524" layer="91"/>
+<wire x1="27.94" y1="27.94" x2="27.94" y2="22.86" width="0.1524" layer="91"/>
+<pinref part="GND7" gate="1" pin="GND"/>
+<wire x1="27.94" y1="22.86" x2="35.56" y2="22.86" width="0.1524" layer="91"/>
 </segment>
 </net>
@@
 <label x="154.94" y="20.32" size="1.778" layer="95"/>
 </segment>
+<segment>
+<pinref part="JP2" gate="A" pin="1"/>
+<wire x1="127" y1="83.82" x2="127" y2="73.66" width="0.1524" layer="91"/>
+<wire x1="127" y1="73.66" x2="116.84" y2="73.66" width="0.1524" layer="91"/>
+<label x="109.22" y="73.66" size="1.778" layer="95"/>
+</segment>
 </net>
 <net name="N$2" class="0">
@@
 <label x="210.82" y="20.32" size="1.778" layer="95"/>
 </segment>
+<segment>
+<pinref part="JP2" gate="A" pin="5"/>
+<wire x1="137.16" y1="83.82" x2="137.16" y2="78.74" width="0.1524" layer="91"/>
+<wire x1="137.16" y1="78.74" x2="147.32" y2="78.74" width="0.1524" layer="91"/>
+<label x="147.32" y="78.74" size="1.778" layer="95"/>
+</segment>
 </net>
 <net name="N$4" class="0">
@@
 <net name="IN+" class="0">
 <segment>
-<pinref part="JP2" gate="G$1" pin="1"/>
 <label x="124.46" y="66.04" size="1.778" layer="95"/>
 <pinref part="U3" gate="A" pin="+IN_B"/>
-<wire x1="129.54" y1="76.2" x2="129.54" y2="40.64" width="0.1524" layer="91"/>
+<wire x1="129.54" y1="76.2" x2="129.54" y2="73.66" width="0.1524" layer="91"/>
+<wire x1="129.54" y1="73.66" x2="129.54" y2="40.64" width="0.1524" layer="91"/>
 <wire x1="129.54" y1="40.64" x2="157.48" y2="40.64" width="0.1524" layer="91"/>
+<pinref part="JP2" gate="A" pin="2"/>
+<wire x1="129.54" y1="83.82" x2="129.54" y2="76.2" width="0.1524" layer="91"/>
 </segment>
 </net>
 <net name="IN-" class="0">
 <segment>
-<pinref part="JP2" gate="G$1" pin="2"/>
-<wire x1="132.08" y1="76.2" x2="132.08" y2="50.8" width="0.1524" layer="91"/>
+<wire x1="132.08" y1="76.2" x2="132.08" y2="73.66" width="0.1524" layer="91"/>
 <label x="134.62" y="66.04" size="1.778" layer="95"/>
 <pinref part="U3" gate="A" pin="+IN_A"/>
+<wire x1="132.08" y1="73.66" x2="132.08" y2="50.8" width="0.1524" layer="91"/>
 <wire x1="132.08" y1="50.8" x2="157.48" y2="50.8" width="0.1524" layer="91"/>
-</segment>
-</net>
+<pinref part="JP2" gate="A" pin="3"/>
+<wire x1="132.08" y1="83.82" x2="132.08" y2="76.2" width="0.1524" layer="91"/>
+</segment>
+</net>

Commit message: Added Board files for instrumentation amplifier
Parts:
- renumbered U1 to VREG+, U2 to VREG-, U3 to OP_AMPS, VR1 to VR+, VR2 to VR-, VR3 to VRAMP
